File: archive_project/archive_test_project.sch (KiCad schematic (older format))
At the start: 5 parts, among them J1 Conn_01x02, J2 Conn_01x02, J3 Screw_Terminal_01x02, U1 LM318J

Commit message: Updated symbols due to library changes
Parts:
- J3: symbol Connector_Specialized:Screw_Terminal_01x02 -> Connector:Screw_Terminal_01x02
Changed lines of the file:
@@
 $EndComp
 $Comp
-L Connector_Specialized:Screw_Terminal_01x02 J3
+L Connector:Screw_Terminal_01x02 J3
 U 1 1 5ABA6E1A
 P 4950 2850
