File: replicate_layout/multiple_hierarchy/test_multiple_hierarchy_top.kicad_pcb (KiCad board)
At the start: 2 copper layers, 64 parts, among them J1001 Pusa_4mm, J1002 Pusa_4mm, J201 Pusa_4mm, J202 Pusa_4mm, J601 Pusa_4mm, J602 Pusa_4mm, Q1101 CSD19531KCS, Q1102 CSD19531KCS, Q1301 CSD19531KCS, Q1302 CSD19531KCS, Q301 CSD19531KCS, Q302 CSD19531KCS, Q501 CSD19531KCS, Q502 CSD19531KCS, Q701 CSD19531KCS, Q702 CSD19531KCS, Q901 CSD19531KCS, Q902 CSD19531KCS, U101 TMS320F28027DA, U1101 IR2181, U1201 INA240, U1301 IR2181, U301 IR2181, U401 INA240, U501 IR2181, U701 IR2181, U801 INA240, U901 IR2181

Commit message: Modified test layout
Parts:
- moved U101 75.7 mm to (91.1, 91.2)
Changed lines of the file:
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@@
   )
   (module Package_SO:TSSOP-38_4.4x9.7mm_P0.5mm (layer F.Cu)
-    (at 155.440001 130.935001)
+    (at 91.059 91.186)
     (descr "TSSOP38: plastic thin shrink small outline package; 38 leads; body width 4.4 mm (see NXP SSOP-TSSOP-VSO-REFLOW.pdf and sot510-1_po.pdf)")
     (tags "SSOP 0.5")
