File: replicate_layout/multiple_hierarchy/multiple_hierarchy_outer.kicad_pcb (KiCad board)
At the start: 2 copper layers, 64 parts, among them J1001 Pusa_4mm, J1002 Pusa_4mm, J201 Pusa_4mm, J202 Pusa_4mm, J601 Pusa_4mm, J602 Pusa_4mm, Q1101 CSD19531KCS, Q1102 CSD19531KCS, Q1301 CSD19531KCS, Q1302 CSD19531KCS, Q301 CSD19531KCS, Q302 CSD19531KCS, Q501 CSD19531KCS, Q502 CSD19531KCS, Q701 CSD19531KCS, Q702 CSD19531KCS, Q901 CSD19531KCS, Q902 CSD19531KCS, U101 TMS320F28027DA, U1101 IR2181, U1201 INA240, U1301 IR2181, U301 IR2181, U401 INA240, U501 IR2181, U701 IR2181, U801 INA240, U901 IR2181

Commit message: Working V2 revision
Parts:
- added C1401: 100n, Passives:C1206M, F.Cu at (181.0, 51.4)
- added C1402: 100n, Passives:C1206M, F.Cu at (184.8, 46.4)
- added D1401: LL4148, Discretes:D_MiniMELF, F.Cu at (181.0, 45.7)
- added Q1401: CSD19531KCS, Discretes:TO-220, F.Cu at (185.4, 33.7)
- added Q1402: CSD19531KCS, Discretes:TO-220, F.Cu at (188.0, 38.7)
- added R1401: 22R, Passives:R1206M, F.Cu at (185.4, 42.5)
- added R1402: 22R, Passives:R1206M, F.Cu at (189.2, 43.2)
- added U1401: IR2181, Package_SO:SO8, F.Cu at (185.4, 51.4)
- moved Q1101 184.0 mm to (31.1, 66.7), turned to 45 degrees
- moved Q1301 96.7 mm to (156.2, 118.1), turned to 45 degrees
- moved J202 71.8 mm to (116.2, 28.6)
- moved Q901 70.6 mm to (148.6, 54.6), turned to 45 degrees
- moved Q701 39.3 mm to (189.9, 100.3)
- moved Q1102 34.6 mm to (222.9, 60.3)
- moved C501 3.65 mm to (110.2, 73.0)
- moved U501 3.65 mm to (111.5, 67.3)
- moved C502 3.65 mm to (110.9, 61.6)
- moved D501 3.65 mm to (107.1, 67.3)
- moved Q501 3.65 mm to (107.1, 53.3)
- moved Q502 3.65 mm to (117.9, 53.3)
- moved R501 3.65 mm to (107.1, 57.8)
- moved R502 3.65 mm to (117.9, 57.8)
- moved J1002 3.16 mm to (190.5, 81.3)
Connections:
- U101 pad 10: Net-(U101-Pad10) -> /Power_extra/Ql
- U101 pad 9: Net-(U101-Pad9) -> /Power_extra/QH
Routing:
- net -VDC: track 65.3 -> 94.1 mm
- net /Leg1/Power-/OUT: track 27.4 -> 46.5 mm
- net /Power_extra/OUT: track 0.00 -> 17.5 mm
- net Net-(R1402-Pad1): track 0.00 -> 12.8 mm
- net +15V: track 27.6 -> 38.0 mm
- net Net-(Q1401-Pad1): track 0.00 -> 7.39 mm
- net Net-(C1402-Pad1): track 0.00 -> 5.82 mm
- net Net-(R1401-Pad1): track 0.00 -> 4.95 mm
- net Net-(Q1402-Pad1): track 0.00 -> 4.54 mm
Other:
- board text added: "A"

Commit message: Updated test projects
Routing:
- net -VDC: track 94.1 -> 94.4 mm, vias 0 -> 4
Changed lines of the file:
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@@
-(kicad_pcb (version 20171130) (host pcbnew "(6.0.0-rc1-dev-1691-g44cb979e9)")
+(kicad_pcb (version 20171130) (host pcbnew "(5.1.2)-1")
   (general
     (thickness 1.6)
-    (drawings 0)
-    (tracks 133)
+    (drawings 1)
+    (tracks 144)
     (zones 0)
     (modules 72)
@@
   (segment (start 112.155 72.62) (end 111.75 73.025) (width 0.5) (layer F.Cu) (net 14))
   (segment (start 114.695 66.04) (end 112.155 68.58) (width 0.5) (layer F.Cu) (net 14))
-  (segment (start 114.695 59.055) (end 114.695 66.04) (width 0.5) (layer F.Cu) (net 14))
   (segment (start 112.155 68.58) (end 112.155 68.735) (width 0.5) (layer F.Cu) (net 14))
   (segment (start 112.155 68.735) (end 112.155 70.01) (width 0.5) (layer F.Cu) (net 14))
@@
   (segment (start 84.795 41.57) (end 86.77 41.57) (width 0.4) (layer F.Cu) (net 14))
   (segment (start 83.495 42.87) (end 84.795 41.57) (width 0.4) (layer F.Cu) (net 14))
-  (segment (start 101.6 53.34) (end 101.6 57.15) (width 0.5) (layer F.Cu) (net 14))
-  (segment (start 101.6 57.15) (end 100.965 57.785) (width 0.5) (layer F.Cu) (net 14))
-  (segment (start 100.965 57.785) (end 94.615 57.785) (width 0.5) (layer F.Cu) (net 14))
-  (segment (start 94.615 57.785) (end 93.345 59.055) (width 0.5) (layer F.Cu) (net 14))
-  (segment (start 90.805 68.735) (end 90.805 70.01) (width 0.5) (layer F.Cu) (net 14))
-  (segment (start 90.805 68.58) (end 90.805 68.735) (width 0.5) (layer F.Cu) (net 14))
-  (segment (start 93.345 59.055) (end 93.345 66.04) (width 0.5) (layer F.Cu) (net 14))
-  (segment (start 93.345 66.04) (end 90.805 68.58) (width 0.5) (layer F.Cu) (net 14))
   (segment (start 90.805 72.62) (end 90.4 73.025) (width 0.5) (layer F.Cu) (net 14))
   (segment (start 90.805 70.01) (end 90.805 72.62) (width 0.5) (layer F.Cu) (net 14))
@@
   (segment (start 186.055 54.135) (end 186.055 53.66) (width 0.5) (layer F.Cu) (net 14))
   (segment (start 186.055 53.66) (end 185.255 52.86) (width 0.5) (layer F.Cu) (net 14))
+  (segment (start 90.805 68.735) (end 90.805 70.01) (width 0.5) (layer F.Cu) (net 14))
+  (segment (start 94.615 57.785) (end 93.345 59.055) (width 0.5) (layer F.Cu) (net 14))
+  (segment (start 90.805 68.58) (end 90.805 68.735) (width 0.5) (layer F.Cu) (net 14))
+  (segment (start 101.6 57.15) (end 100.965 57.785) (width 0.5) (layer F.Cu) (net 14))
+  (segment (start 101.6 53.34) (end 101.6 57.15) (width 0.5) (layer F.Cu) (net 14))
+  (segment (start 100.965 57.785) (end 94.615 57.785) (width 0.5) (layer F.Cu) (net 14))
+  (segment (start 93.345 66.04) (end 90.805 68.58) (width 0.5) (layer F.Cu) (net 14))
+  (via (at 93.345 64.77) (size 0.8) (drill 0.4) (layers F.Cu B.Cu) (net 14))
+  (segment (start 93.345 66.04) (end 93.345 64.77) (width 0.25) (layer F.Cu) (net 14))
+  (via (at 93.345 59.69) (size 0.8) (drill 0.4) (layers F.Cu B.Cu) (net 14))
+  (segment (start 93.345 64.77) (end 93.345 59.69) (width 0.25) (layer B.Cu) (net 14))
+  (segment (start 93.345 59.69) (end 93.345 59.055) (width 0.25) (layer F.Cu) (net 14))
+  (via (at 114.935 64.77) (size 0.8) (drill 0.4) (layers F.Cu B.Cu) (net 14))
+  (segment (start 114.695 66.04) (end 114.695 65.01) (width 0.25) (layer F.Cu) (net 14))
+  (segment (start 114.695 65.01) (end 114.935 64.77) (width 0.25) (layer F.Cu) (net 14))
+  (via (at 114.935 59.69) (size 0.8) (drill 0.4) (layers F.Cu B.Cu) (net 14))
+  (segment (start 114.935 64.77) (end 114.935 59.69) (width 0.25) (layer B.Cu) (net 14))
+  (segment (start 114.865685 59.055) (end 114.695 59.055) (width 0.25) (layer F.Cu) (net 14))
+  (segment (start 114.935 59.124315) (end 114.865685 59.055) (width 0.25) (layer F.Cu) (net 14))
+  (segment (start 114.935 59.69) (end 114.935 59.124315) (width 0.25) (layer F.Cu) (net 14))
   (segment (start 87.025 59.285) (end 85.725 59.285) (width 0.5) (layer F.Cu) (net 17))
   (segment (start 87.835002 59.285) (end 87.025 59.285) (width 0.5) (layer F.Cu) (net 17))
