File: replicate_layout/multiple_hierarchy/multiple_hierarchy_outer_test.kicad_pcb (KiCad board)
At the start: 2 copper layers, 72 parts, among them J1001 Pusa_4mm, J1002 Pusa_4mm, J201 Pusa_4mm, J202 Pusa_4mm, J601 Pusa_4mm, J602 Pusa_4mm, Q1101 CSD19531KCS, Q1102 CSD19531KCS, Q1301 CSD19531KCS, Q1302 CSD19531KCS, Q1401 CSD19531KCS, Q1402 CSD19531KCS, Q301 CSD19531KCS, Q302 CSD19531KCS, Q501 CSD19531KCS, Q502 CSD19531KCS, Q701 CSD19531KCS, Q702 CSD19531KCS, Q901 CSD19531KCS, Q902 CSD19531KCS, U101 TMS320F28027DA, U1101 IR2181, U1201 INA240, U1301 IR2181, U1401 IR2181, U301 IR2181, U401 INA240, U501 IR2181, U701 IR2181, U801 INA240, U901 IR2181

Commit message: Updated test projects
Routing:
- net -VDC: track 159.5 -> 160.1 mm, vias 0 -> 8
