File: archive_project/archived_test_project/archive_test_project.sch (KiCad schematic (older format))
At the start: 5 parts, among them J1 Conn_01x02, J2 Conn_01x02, J3 Screw_Terminal_01x02, U1 LM318J

Commit message: Updated test project
Parts:
- removed U1: LM318J, Package_DIP:DIP-14_W7.62mm, symbol archive:Amplifier_Operational_LM318J
- added U101: LM318J, Package_DIP:DIP-14_W7.62mm, symbol archive:Amplifier_Operational_LM318J
Connections:
- net +15V: now also U101.11 (V+)
- net GND: now also U101.6 (V-)
- net subsheet/IN: now also U101.10, U101.4 (-)
- net at J1.2 (Pin_2): now also U101.5 (+)
Changed lines of the file:
@@
 EESchema Schematic File Version 4
-LIBS:archive_test_project-cache
 EELAYER 29 0
 EELAYER END
@@
 $EndSheet
 $Comp
-L archive:Amplifier_Operational_LM318J U1
-U 1 1 5ABA5C92
-P 2750 2850
-F 0 "U1" H 2850 3100 50  0000 L CNN
-F 1 "LM318J" H 2850 3000 50  0000 L CNN
-F 2 "Package_DIP:DIP-14_W7.62mm" H 2750 2850 50  0001 C CNN
-F 3 "http://www.ti.com/lit/ds/symlink/lm318-n.pdf" H 2750 2850 50  0001 C CNN
-	1    2750 2850
-	1    0    0    -1
-$EndComp
-$Comp
 L archive:power_GND #PWR05
 U 1 1 5ABA5CE0
@@
 F1 "hiearchical_sub/file5ACC74AA.sch" 50
 $EndSheet
+$Comp
+L archive:Amplifier_Operational_LM318J U101
+U 1 1 5C8821F3
+P 2750 2850
+F 0 "U101" H 2900 3000 50  0000 L CNN
+F 1 "LM318J" H 2900 2700 50  0000 L CNN
+F 2 "Package_DIP:DIP-14_W7.62mm" H 2750 2850 50  0001 C CNN
+F 3 "http://www.ti.com/lit/ds/symlink/lm318-n.pdf" H 2750 2850 50  0001 C CNN
+	1    2750 2850
+	1    0    0    -1
+$EndComp
 $EndSCHEMATC
