File: copy_layout/Source_project/multiple_hierarchy.kicad_pcb (KiCad board)
At the start: 2 copper layers, 72 parts, among them J1001 Pusa_4mm, J1002 Pusa_4mm, J201 Pusa_4mm, J202 Pusa_4mm, J601 Pusa_4mm, J602 Pusa_4mm, Q1101 CSD19531KCS, Q1102 CSD19531KCS, Q1301 CSD19531KCS, Q1302 CSD19531KCS, Q1401 CSD19531KCS, Q1402 CSD19531KCS, Q301 CSD19531KCS, Q302 CSD19531KCS, Q501 CSD19531KCS, Q502 CSD19531KCS, Q701 CSD19531KCS, Q702 CSD19531KCS, Q901 CSD19531KCS, Q902 CSD19531KCS, U101 TMS320F28027DA, U1101 IR2181, U1201 INA240, U1301 IR2181, U1401 IR2181, U301 IR2181, U401 INA240, U501 IR2181, U701 IR2181, U801 INA240, U901 IR2181

Commit message: Delna verzija
Parts:
- moved R501 87.9 mm to (107.3, 57.8), turned to 90 degrees
- moved Q502 81.3 mm to (118.1, 53.3)
- moved C502 79.1 mm to (111.1, 61.6)
- moved R502 77.6 mm to (118.1, 57.8), turned to 90 degrees
- moved D501 76.6 mm to (107.3, 67.3), turned to 270 degrees
- moved J202 72.2 mm to (114.9, 28.6)
- moved C501 71.3 mm to (110.5, 73.0)
- moved U501 70.1 mm to (111.8, 67.3), turned to 90 degrees
Routing:
- net /Leg1/Power-/OUT: track 0.00 -> 47.0 mm
- net -VDC: track 66.1 -> 94.1 mm
- net +15V: track 24.2 -> 38.0 mm
- net Net-(R502-Pad1): track 0.00 -> 13.0 mm
- net Net-(R501-Pad1): track 0.00 -> 8.14 mm
- net Net-(C502-Pad1): track 0.00 -> 6.04 mm
- net Net-(Q502-Pad1): track 0.00 -> 2.94 mm
- net Net-(Q501-Pad1): track 0.00 -> 2.94 mm
- added copper zone on F.Cu, net /Leg1/Power-/OUT
- added copper zone on F.Cu, net /Power_extra/OUT
Other:
- board text added: "tret"
