File: swap_units/swap_units_test_project/Level3.sch (KiCad schematic (older format))
At the start: 5 parts, among them U7 LM324

Commit message: updated test projects
Connections:
- net out_level_2: no longer U7.13 (-), U7.14
- new net out_level_1: U7.13 (-), U7.14
Changed lines of the file:
@@
 	3550 4300 3400 4300
 Text HLabel 3550 4300 2    50   Output ~ 0
-out_level_2
+out_level_1
 $Comp
 L Amplifier_Operational:LM324 U7
