File: swap_units/swap_units_test_project_different_sheets/swap_units_test.kicad_pcb (KiCad board)
At the start: 2 copper layers, 22 parts, among them U1 LM324, U2 PIC18F452-IP, U3 LM324, U7 LM324, U8 LM324

Commit message: updated test projects
Connections:
- U7 pad 13: /Level1/Level3a/out_level_2 -> /Level1/Level3a/out_level_1
- U7 pad 14: /Level1/Level3a/out_level_2 -> /Level1/Level3a/out_level_1
- U8 pad 13: /Level1/Level3b/out_level_2 -> /Level1/Level3b/out_level_1
- U8 pad 14: /Level1/Level3b/out_level_2 -> /Level1/Level3b/out_level_1
Changed lines of the file:
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@@
     (zones 0)
     (modules 22)
-    (nets 54)
+    (nets 56)
   )
   (page A4)
@@
   (net 52 /Level1/Level3a/out_level_2)
   (net 53 /Level1/Level3b/out_level_2)
+  (net 54 /Level1/Level3a/out_level_1)
+  (net 55 /Level1/Level3b/out_level_1)
   (net_class Default "This is the default net class."
     (clearance 0.2)
@@
     (add_net +5V)
     (add_net /Level1/Level2b/out_level_2)
+    (add_net /Level1/Level3a/out_level_1)
     (add_net /Level1/Level3a/out_level_2)
+    (add_net /Level1/Level3b/out_level_1)
     (add_net /Level1/Level3b/out_level_2)
     (add_net /Level1/out_level_1)
@@
     (fp_arc (start 3.81 -1.33) (end 2.81 -1.33) (angle -180) (layer F.SilkS) (width 0.12))
     (pad 14 thru_hole oval (at 7.62 0) (size 1.6 1.6) (drill 0.8) (layers *.Cu *.Mask)
-      (net 53 /Level1/Level3b/out_level_2))
+      (net 55 /Level1/Level3b/out_level_1))
     (pad 7 thru_hole oval (at 0 15.24) (size 1.6 1.6) (drill 0.8) (layers *.Cu *.Mask)
       (net 53 /Level1/Level3b/out_level_2))
     (pad 13 thru_hole oval (at 7.62 2.54) (size 1.6 1.6) (drill 0.8) (layers *.Cu *.Mask)
-      (net 53 /Level1/Level3b/out_level_2))
+      (net 55 /Level1/Level3b/out_level_1))
     (pad 6 thru_hole oval (at 0 12.7) (size 1.6 1.6) (drill 0.8) (layers *.Cu *.Mask)
       (net 53 /Level1/Level3b/out_level_2))
@@
     (fp_arc (start 3.81 -1.33) (end 2.81 -1.33) (angle -180) (layer F.SilkS) (width 0.12))
     (pad 14 thru_hole oval (at 7.62 0) (size 1.6 1.6) (drill 0.8) (layers *.Cu *.Mask)
-      (net 52 /Level1/Level3a/out_level_2))
+      (net 54 /Level1/Level3a/out_level_1))
     (pad 7 thru_hole oval (at 0 15.24) (size 1.6 1.6) (drill 0.8) (layers *.Cu *.Mask)
       (net 52 /Level1/Level3a/out_level_2))
     (pad 13 thru_hole oval (at 7.62 2.54) (size 1.6 1.6) (drill 0.8) (layers *.Cu *.Mask)
-      (net 52 /Level1/Level3a/out_level_2))
+      (net 54 /Level1/Level3a/out_level_1))
     (pad 6 thru_hole oval (at 0 12.7) (size 1.6 1.6) (drill 0.8) (layers *.Cu *.Mask)
       (net 52 /Level1/Level3a/out_level_2))
