File: swap_units/swap_units_test_project_same_sheet_different_hierarchy/swap_units_test.kicad_pcb (KiCad board)
At the start: 2 copper layers, 22 parts, among them U1 LM324, U2 PIC18F452-IP, U3 LM324, U7 LM324, U8 LM324

Commit message: updated reference test projects
Connections:
- U1 pad 10: Net-(R6-Pad2) -> Net-(R4-Pad2)
- U1 pad 12: Net-(R4-Pad2) -> Net-(R6-Pad2)
- U1 pad 13: /Level1/out_level_1 -> /Level1/out_level_2
- U1 pad 14: /Level1/out_level_1 -> /Level1/out_level_2
- U1 pad 8: /Level1/out_level_2 -> /Level1/out_level_1
- U1 pad 9: /Level1/out_level_2 -> /Level1/out_level_1
- U3 pad 1: /Level1/Level2b/out_level_2 -> Net-(U3-Pad1)
- U3 pad 12: Net-(U3-Pad3) -> Net-(R8-Pad2)
- U3 pad 13: Net-(U3-Pad2) -> /Level1/Level2b/out_level_2
- U3 pad 14: Net-(U3-Pad1) -> /Level1/Level2b/out_level_2
- U3 pad 2: /Level1/Level2b/out_level_2 -> Net-(U3-Pad2)
- U3 pad 3: Net-(R8-Pad2) -> Net-(U3-Pad3)
Changed lines of the file:
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@@
     (fp_arc (start 3.81 -1.33) (end 2.81 -1.33) (angle -180) (layer F.SilkS) (width 0.12))
     (pad 14 thru_hole oval (at 7.62 0) (size 1.6 1.6) (drill 0.8) (layers *.Cu *.Mask)
-      (net 47 "Net-(U3-Pad1)"))
+      (net 44 /Level1/Level2b/out_level_2))
     (pad 7 thru_hole oval (at 0 15.24) (size 1.6 1.6) (drill 0.8) (layers *.Cu *.Mask))
     (pad 13 thru_hole oval (at 7.62 2.54) (size 1.6 1.6) (drill 0.8) (layers *.Cu *.Mask)
-      (net 46 "Net-(U3-Pad2)"))
+      (net 44 /Level1/Level2b/out_level_2))
     (pad 6 thru_hole oval (at 0 12.7) (size 1.6 1.6) (drill 0.8) (layers *.Cu *.Mask))
     (pad 12 thru_hole oval (at 7.62 5.08) (size 1.6 1.6) (drill 0.8) (layers *.Cu *.Mask)
-      (net 45 "Net-(U3-Pad3)"))
+      (net 43 "Net-(R8-Pad2)"))
     (pad 5 thru_hole oval (at 0 10.16) (size 1.6 1.6) (drill 0.8) (layers *.Cu *.Mask))
     (pad 11 thru_hole oval (at 7.62 7.62) (size 1.6 1.6) (drill 0.8) (layers *.Cu *.Mask))
@@
     (pad 10 thru_hole oval (at 7.62 10.16) (size 1.6 1.6) (drill 0.8) (layers *.Cu *.Mask))
     (pad 3 thru_hole oval (at 0 5.08) (size 1.6 1.6) (drill 0.8) (layers *.Cu *.Mask)
-      (net 43 "Net-(R8-Pad2)"))
+      (net 45 "Net-(U3-Pad3)"))
     (pad 9 thru_hole oval (at 7.62 12.7) (size 1.6 1.6) (drill 0.8) (layers *.Cu *.Mask))
     (pad 2 thru_hole oval (at 0 2.54) (size 1.6 1.6) (drill 0.8) (layers *.Cu *.Mask)
-      (net 44 /Level1/Level2b/out_level_2))
+      (net 46 "Net-(U3-Pad2)"))
     (pad 8 thru_hole oval (at 7.62 15.24) (size 1.6 1.6) (drill 0.8) (layers *.Cu *.Mask))
     (pad 1 thru_hole rect (at 0 0) (size 1.6 1.6) (drill 0.8) (layers *.Cu *.Mask)
-      (net 44 /Level1/Level2b/out_level_2))
+      (net 47 "Net-(U3-Pad1)"))
     (model ${KISYS3DMOD}/Package_DIP.3dshapes/DIP-14_W7.62mm.wrl
       (at (xyz 0 0 0))
@@
       (net 7 "Net-(U1-Pad1)"))
     (pad 8 thru_hole oval (at 7.62 15.24) (size 1.6 1.6) (drill 0.8) (layers *.Cu *.Mask)
-      (net 10 /Level1/out_level_2))
+      (net 8 /Level1/out_level_1))
     (pad 2 thru_hole oval (at 0 2.54) (size 1.6 1.6) (drill 0.8) (layers *.Cu *.Mask)
       (net 7 "Net-(U1-Pad1)"))
     (pad 9 thru_hole oval (at 7.62 12.7) (size 1.6 1.6) (drill 0.8) (layers *.Cu *.Mask)
-      (net 10 /Level1/out_level_2))
+      (net 8 /Level1/out_level_1))
     (pad 3 thru_hole oval (at 0 5.08) (size 1.6 1.6) (drill 0.8) (layers *.Cu *.Mask)
       (net 2 "Net-(R1-Pad2)"))
     (pad 10 thru_hole oval (at 7.62 10.16) (size 1.6 1.6) (drill 0.8) (layers *.Cu *.Mask)
-      (net 6 "Net-(R6-Pad2)"))
+      (net 5 "Net-(R4-Pad2)"))
     (pad 4 thru_hole oval (at 0 7.62) (size 1.6 1.6) (drill 0.8) (layers *.Cu *.Mask)
       (net 1 +5V))
@@
       (net 3 "Net-(R2-Pad2)"))
     (pad 12 thru_hole oval (at 7.62 5.08) (size 1.6 1.6) (drill 0.8) (layers *.Cu *.Mask)
-      (net 5 "Net-(R4-Pad2)"))
+      (net 6 "Net-(R6-Pad2)"))
     (pad 6 thru_hole oval (at 0 12.7) (size 1.6 1.6) (drill 0.8) (layers *.Cu *.Mask)
       (net 9 "Net-(U1-Pad6)"))
     (pad 13 thru_hole oval (at 7.62 2.54) (size 1.6 1.6) (drill 0.8) (layers *.Cu *.Mask)
-      (net 8 /Level1/out_level_1))
+      (net 10 /Level1/out_level_2))
     (pad 7 thru_hole oval (at 0 15.24) (size 1.6 1.6) (drill 0.8) (layers *.Cu *.Mask)
       (net 9 "Net-(U1-Pad6)"))
     (pad 14 thru_hole oval (at 7.62 0) (size 1.6 1.6) (drill 0.8) (layers *.Cu *.Mask)
-      (net 8 /Level1/out_level_1))
+      (net 10 /Level1/out_level_2))
     (model ${KISYS3DMOD}/Package_DIP.3dshapes/DIP-14_W7.62mm.wrl
       (at (xyz 0 0 0))

Commit message: updated test projects
Connections:
- U7 pad 6: /Level1/Level3a/out_level_2 -> /Level1/Level3a/out_level_1
- U7 pad 7: /Level1/Level3a/out_level_2 -> /Level1/Level3a/out_level_1
- U8 pad 13: /Level1/Level3b/out_level_2 -> /Level1/Level3b/out_level_1
- U8 pad 14: /Level1/Level3b/out_level_2 -> /Level1/Level3b/out_level_1
Changed lines of the file:
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@@
     (zones 0)
     (modules 22)
-    (nets 54)
+    (nets 56)
   )
   (page A4)
@@
   (net 52 /Level1/Level3a/out_level_2)
   (net 53 /Level1/Level3b/out_level_2)
+  (net 54 /Level1/Level3a/out_level_1)
+  (net 55 /Level1/Level3b/out_level_1)
   (net_class Default "This is the default net class."
     (clearance 0.2)
@@
     (add_net +5V)
     (add_net /Level1/Level2b/out_level_2)
+    (add_net /Level1/Level3a/out_level_1)
     (add_net /Level1/Level3a/out_level_2)
+    (add_net /Level1/Level3b/out_level_1)
     (add_net /Level1/Level3b/out_level_2)
     (add_net /Level1/out_level_1)
@@
     (fp_arc (start 3.81 -1.33) (end 2.81 -1.33) (angle -180) (layer F.SilkS) (width 0.12))
     (pad 14 thru_hole oval (at 7.62 0) (size 1.6 1.6) (drill 0.8) (layers *.Cu *.Mask)
-      (net 53 /Level1/Level3b/out_level_2))
+      (net 55 /Level1/Level3b/out_level_1))
     (pad 7 thru_hole oval (at 0 15.24) (size 1.6 1.6) (drill 0.8) (layers *.Cu *.Mask)
       (net 53 /Level1/Level3b/out_level_2))
     (pad 13 thru_hole oval (at 7.62 2.54) (size 1.6 1.6) (drill 0.8) (layers *.Cu *.Mask)
-      (net 53 /Level1/Level3b/out_level_2))
+      (net 55 /Level1/Level3b/out_level_1))
     (pad 6 thru_hole oval (at 0 12.7) (size 1.6 1.6) (drill 0.8) (layers *.Cu *.Mask)
       (net 53 /Level1/Level3b/out_level_2))
@@
       (net 52 /Level1/Level3a/out_level_2))
     (pad 7 thru_hole oval (at 0 15.24) (size 1.6 1.6) (drill 0.8) (layers *.Cu *.Mask)
-      (net 52 /Level1/Level3a/out_level_2))
+      (net 54 /Level1/Level3a/out_level_1))
     (pad 13 thru_hole oval (at 7.62 2.54) (size 1.6 1.6) (drill 0.8) (layers *.Cu *.Mask)
       (net 52 /Level1/Level3a/out_level_2))
     (pad 6 thru_hole oval (at 0 12.7) (size 1.6 1.6) (drill 0.8) (layers *.Cu *.Mask)
-      (net 52 /Level1/Level3a/out_level_2))
+      (net 54 /Level1/Level3a/out_level_1))
     (pad 12 thru_hole oval (at 7.62 5.08) (size 1.6 1.6) (drill 0.8) (layers *.Cu *.Mask)
       (net 48 "Net-(R10-Pad2)"))
