File: save_restore_layout/Destination_project/Destination_project.kicad_pcb (KiCad board)
At the start: 2 copper layers, 51 parts, among them J1 Pusa_4mm, J2 Pusa_4mm, J3 Pusa_4mm, J4 Pusa_4mm, Q1 CSD19531KCS, Q10 CSD19531KCS, Q2 CSD19531KCS, Q3 CSD19531KCS, Q4 CSD19531KCS, Q5 CSD19531KCS, Q6 CSD19531KCS, Q7 CSD19531KCS, Q8 CSD19531KCS, Q9 CSD19531KCS, U1 LAUNCHXL-F28379D, U2 IR2181, U3 IR2181, U4 INA240, U5 IR2181, U6 IR2181, U7 INA240, U8 IR2181

Commit message: Changed test projects
Parts:
- moved Q3 68.0 mm to (104.8, 45.7)
- moved U1 62.1 mm to (-6.99, 77.5)
Changed lines of the file:
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@@
-(kicad_pcb (version 20171130) (host pcbnew "(5.1.0)-1")
+(kicad_pcb (version 20171130) (host pcbnew "(5.1.2)-1")
   (general
     (thickness 1.6)
@@
   )
   (module Module:28379D_launchpad (layer F.Cu)
-    (at 54.838 71.284)
+    (at -6.985 77.47)
     (descr "28379D launchpad")
     (tags DEV)
@@
   )
   (module Discretes:TO-220 (layer F.Cu)
-    (at 172.738 47.224)
+    (at 104.775 45.72)
     (descr "TO-220-3, Vertical, RM 2.54mm")
     (tags "TO-220-3 Vertical RM 2.54mm")
